File: Hardware/untitled1.kicad_sch (KiCad schematic)
At the start: 26 parts, among them J1 Conn_01x03_Pin, J2 Conn_01x02_Pin, J3 Conn_01x03_Pin, J4 Conn_01x06_Pin, J5 Conn_01x03_Pin, J6 Conn_01x03_Socket, SW2 RESET_Btn, U3 PIC32MM0256GPM064-I/PT, U5 W25Q64FVSSIG

Commit message: CHECK
CHECK1
Parts:
- removed J6: Conn_01x03_Socket, symbol Connector:Conn_01x03_Socket
- removed U4: ~, symbol thinh:Conn_02x21__Odd_Even
- added J6: Conn_01x02_Socket, symbol Connector:Conn_01x02_Socket
- added Y1: Crystal, symbol Device:Crystal
Connections:
- net OSC1: now also J6.1 (Pin_1), Y1.2
- net OSC2: now also J6.2 (Pin_2), Y1.1
- net BO_1: no longer names the net of U3.1 (RP21/SDI3/RA7)
- net BO_11 renamed C1IND
- net BO_12: no longer names the net of U3.20 (AN13/T3CK/T3G/RC1)
- net BO_13: no longer names the net of U3.21 (RP19/OCM2A/RC2)
- net BO_14: no longer names the net of U3.22 (SS3/FSYNC3/RC11)
- net BO_17: no longer names the net of U3.27 (SDO3/RA8)
- net BO_18: no longer names the net of U3.28 (SOSCI/AN7/RP10/RB4)
- net BO_19: no longer names the net of U3.29 (SOSCO/SCLKI/RP5/PWRLCLK/RA4)
- net BO_2: no longer names the net of U3.2 (CVREF/AN9/C3INB/RP16/VBUSON/RB14)
- net BO_20: no longer names the net of U3.30 (RP24/RA9)
- net BO_21: no longer names the net of U3.64 (RP22/SCK3/RA10)
- net BO_22: no longer names the net of U3.63 (AN8/RP15/SCL3/RB13)
- net BO_23: no longer names the net of U3.61 (D+/RB11)
- net BO_24: no longer names the net of U3.60 (D-/RB10)
- net BO_25: no longer names the net of U3.59 (OCM3C/RA14)
- net BO_26: no longer names the net of U3.58 (RTCC/RA15)
- net BO_27: no longer names the net of U3.55 (PGEC3/TDO/RP18/ASCL1/USBOEN/RC9)
- net BO_28: no longer names the net of U3.54 (OCM3A/RA5)
- net BO_29: no longer names the net of U3.53 (OCM1B/RD1)
- net BO_3: no longer names the net of U3.3 (AN10/C3INA/REFCLKO/RP17/RB15)
- net BO_30: no longer names the net of U3.52 (AN14/LVDIN/C2INC/RC8)
- net BO_31: no longer names the net of U3.51 (RP20/RC7)
- net BO_34: no longer names the net of U3.46 (RP12/SDA3/RB7)
- net BO_35: no longer names the net of U3.44 (VBUS/RB6)
- net BO_36: no longer names the net of U3.43 (PGED3/RP11/ASDA1/USBID/RB5)
- net BO_37: no longer names the net of U3.42 (OCM3E/RC15)
- net BO_38: no longer names the net of U3.41 (OCM3D/RC14)
- net BO_39: no longer names the net of U3.37 (AN15/OCM1D/RC5)
- net BO_4: no longer names the net of U3.6 (AN16/U1CTS/RA13)
- net BO_40: no longer names the net of U3.36 (OCM1E/INT3/RC4)
- net BO_41: no longer names the net of U3.35 (OCM2B/RC3)
- net BO_42: no longer names the net of U3.33 (OCM3B/RD3)
- net BO_5: no longer names the net of U3.7 (AN17/OCM1A/RA12)
- net BO_6: no longer names the net of U3.8 (AN18/RA11)
- net BO_7 renamed RA0
- net BO_8 renamed RA1
- no-connect marks 1 -> 34
Other:
- note removed: "Pin Breakout"
- moved on the sheet: C25, C26, D4, R12, R4, R5, SW2

Commit message: CHECK
CHECK
Connections:
- net RA8: now reaches U3.27 (SDO3/RA8)
- net RB4: now reaches U3.28 (SOSCI/AN7/RP10/RB4)
- net RA4: now reaches U3.29 (SOSCO/SCLKI/RP5/PWRLCLK/RA4)
- no-connect marks 34 -> 31
Changed lines of the file:
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@@
   (no_connect (at 262.255 55.245))
   (no_connect (at 148.59 70.485))
-  (no_connect (at 148.59 118.745))
   (no_connect (at 148.59 106.045))
-  (no_connect (at 148.59 123.825))
   (no_connect (at 148.59 67.945))
   (no_connect (at 262.255 123.825))
@@
   (no_connect (at 262.255 111.125))
   (no_connect (at 262.255 85.725))
-  (no_connect (at 148.59 121.285))
   (no_connect (at 254 90.805))
   (no_connect (at 148.59 100.965))
@@
     (effects (font (size 1.27 1.27)) (justify left))
   )
+  (hierarchical_label "RA8" (shape input) (at 148.59 118.745 180) (fields_autoplaced)
+    (effects (font (size 1.27 1.27)) (justify right))
+  )
   (hierarchical_label "3V3" (shape input) (at 87.63 55.88 90) (fields_autoplaced)
     (effects (font (size 1.27 1.27)) (justify left))
@@
     (effects (font (size 1.27 1.27)) (justify right))
   )
+  (hierarchical_label "RA4" (shape input) (at 148.59 123.825 180) (fields_autoplaced)
+    (effects (font (size 1.27 1.27)) (justify right))
+  )
   (hierarchical_label "3V3" (shape input) (at 39.37 23.495 90) (fields_autoplaced)
     (effects (font (size 1.27 1.27)) (justify left))
@@
     (effects (font (size 1.27 1.27)) (justify right))
   )
+  (hierarchical_label "RB4" (shape input) (at 148.59 121.285 180) (fields_autoplaced)
+    (effects (font (size 1.27 1.27)) (justify right))
+  )
