File: Hardware/WeatherStation.kicad_pcb (KiCad board)
At the start: 2 copper layers, 73.2 x 82.3 mm, 0 parts

Commit message: UPDATE _FOOTPRINT
UPDATE
Parts:
- added ANT1: 0.9-1.8GHz, SAMPI:AH3G.303, F.Cu at (246.9, 42.6)
- added ANT2: UFL, SAMPI:U.FL, F.Cu at (87.7, 95.5)
- added BAT1: 3.7V/1.8Ah, SAMPI:BAT18650-PCBPAD, B.Cu at (230.2, 87.3)
- added BAT2: 3.7V/1.8Ah, SAMPI:BAT18650-PCBPAD, B.Cu at (230.3, 68.5)
- added BT1: RESET, SAMPI:SW_SMD2_6.0x3.5, F.Cu at (120.7, 44.1)
- added BT2: APP, SAMPI:SW_SMD2_6.0x3.5, F.Cu at (120.7, 49.1)
- added C1: 100nF, SAMPI:CAP0603, F.Cu at (58.0, 103.4)
- added C10: 100pF, SAMPI:CAP0603, F.Cu at (58.0, 116.4)
- added C11: 100pF, SAMPI:CAP0603, F.Cu at (58.0, 119.0)
- added C12: 100nF, SAMPI:CAP0603, F.Cu at (58.0, 121.6)
- added C13: 100pF, SAMPI:CAP0603, F.Cu at (61.7, 103.4)
- added C14: 10uF, SAMPI:CAP0805, F.Cu at (65.5, 133.5)
- added C15: 100pF, SAMPI:CAP0603, F.Cu at (61.7, 106.0)
- added C16: 100nF, SAMPI:CAP0603, F.Cu at (61.7, 108.6)
- added C17: 100nF, SAMPI:CAP0603, F.Cu at (61.7, 111.2)
- added C18: 10uF, SAMPI:CAP0805, F.Cu at (65.5, 136.5)
- added C19: 220uF, SAMPI:CAP2312-6032, F.Cu at (79.3, 114.7)
- added C2: 10uF, SAMPI:CAP0805, F.Cu at (65.5, 124.5)
- added C20: 220uF, SAMPI:CAP2312-6032, F.Cu at (48.6, 108.2)
- added C21: 10uF, SAMPI:CAP0805, F.Cu at (69.4, 124.5)
- added C22: 10uF, SAMPI:CAP0805, F.Cu at (69.4, 127.5)
- added C23: 100pF, SAMPI:CAP0603, F.Cu at (61.7, 113.8)
- added C24: 10uF, SAMPI:CAP0805, F.Cu at (69.4, 130.5)
- added C25: 100nF, SAMPI:CAP0603, F.Cu at (61.7, 116.4)
- added C26: 220uF, SAMPI:CAP2312-6032, F.Cu at (48.6, 120.5)
- added C27: 100nF, SAMPI:CAP0603, F.Cu at (107.0, 42.9)
- added C28: 8.2pF, SAMPI:CAP0603, F.Cu at (107.0, 45.5)
- added C29: 8.2pF, SAMPI:CAP0603, F.Cu at (107.0, 48.1)
- added C3: 10uF, SAMPI:CAP0805, F.Cu at (65.5, 127.5)
- added C30: 10uF, SAMPI:CAP0805, F.Cu at (124.9, 56.2)
- added C31: 2.2uF, SAMPI:CAP0603, F.Cu at (107.0, 50.8)
- added C32: 22pF, SAMPI:CAP0603, F.Cu at (107.0, 53.4)
- added C33: 22pF, SAMPI:CAP0603, F.Cu at (107.0, 56.0)
- added C34: 100nF, SAMPI:CAP0603, F.Cu at (110.8, 42.9)
- added C35: 22pF, SAMPI:CAP0603, F.Cu at (110.8, 45.5)
- added C36: 2.2uF, SAMPI:CAP0603, F.Cu at (110.8, 48.1)
- added C37: 22pF, SAMPI:CAP0603, F.Cu at (110.8, 50.8)
- added C38: 22pF, SAMPI:CAP0603, F.Cu at (72.0, 75.9)
- added C39: 22pF, SAMPI:CAP0603, F.Cu at (72.0, 78.5)
- added C4: 100pF, SAMPI:CAP0603, F.Cu at (58.0, 106.0)
- added C40: 22pF, SAMPI:CAP0603, F.Cu at (72.0, 81.1)
- added C41: 100nF, SAMPI:CAP0603, F.Cu at (72.0, 83.7)
- added C42: 100nF, SAMPI:CAP0603, F.Cu at (72.0, 86.3)
- added C43: 22pF, SAMPI:CAP0603, F.Cu at (72.0, 88.9)
- added C44: 2.2uF, SAMPI:CAP0603, F.Cu at (72.0, 91.5)
- added C45: 22pF, SAMPI:CAP0603, F.Cu at (72.0, 94.2)
- added C46: 100nF, SAMPI:CAP0603, F.Cu at (75.7, 75.9)
- added C47: 100nF, SAMPI:CAP0603, F.Cu at (75.7, 78.5)
- added C48: 22pF, SAMPI:CAP0603, F.Cu at (75.7, 81.1)
- added C49: 220uF, SAMPI:CAP2312-6032, F.Cu at (89.6, 84.3)
- added C5: 470uF, SAMPI:CAP_ELEC-10.3x10.3-DIA10, F.Cu at (79.3, 106.3)
- added C50: 2.2uF, SAMPI:CAP0603, F.Cu at (75.7, 83.7)
- added C51: 100nF, SAMPI:CAP0603, F.Cu at (75.7, 86.3)
- added C52: 22pF, SAMPI:CAP0603, F.Cu at (75.7, 88.9)
- added C53: 22pF, SAMPI:CAP0603, F.Cu at (75.7, 91.5)
- added C54: 22pF, SAMPI:CAP0603, F.Cu at (75.7, 94.2)
- added C55: 2.2uF, SAMPI:CAP0603, F.Cu at (79.4, 75.9)
- added C56: 22pF, SAMPI:CAP0603, F.Cu at (79.4, 78.5)
- added C57: 10F/2.7V, SAMPI:SCAP1320, F.Cu at (223.4, 83.2)
- added C58: 10F/2.7V, SAMPI:SCAP1320, F.Cu at (223.3, 68.4)
- added C59: 22pF, SAMPI:CAP0603, F.Cu at (79.4, 81.1)
- added C6: 100nF, SAMPI:CAP0603, F.Cu at (58.0, 108.6)
- added C60: 2.2uF, SAMPI:CAP0603, F.Cu at (79.4, 83.7)
- added C61: 100nF, SAMPI:CAP0603, F.Cu at (79.4, 86.3)
- added C62: 10uF, SAMPI:CAP0805, F.Cu at (99.7, 90.0)
- added C63: 10uF, SAMPI:CAP0805, F.Cu at (252.4, 129.3)
- added C64: 10uF, SAMPI:CAP0805, F.Cu at (108.5, 106.6)
- added C65: 220uF, SAMPI:CAP2312-6032, F.Cu at (234.7, 132.0)
- added C66: 100nF, SAMPI:CAP0603, F.Cu at (241.2, 129.1)
- added C67: 10uF, SAMPI:CAP0805, F.Cu at (252.4, 135.3)
- added C68: 100pF, SAMPI:CAP0603, F.Cu at (97.3, 106.0)
- added C69: 100pF, SAMPI:CAP0603, F.Cu at (241.2, 134.3)
- added C7: 10uF, SAMPI:CAP0805, F.Cu at (65.5, 130.5)
- added C70: 100nF, SAMPI:CAP0603, F.Cu at (97.3, 111.2)
- added C71: 22pF, SAMPI:CAP0603, F.Cu at (97.3, 113.8)
- added C72: 220uF, SAMPI:CAP2312-6032, F.Cu at (90.8, 114.7)
- added C73: 22pF, SAMPI:CAP0603, F.Cu at (101.0, 103.4)
- added C74: 100nF, SAMPI:CAP0603, F.Cu at (256.1, 120.0)
- added C75: 10uF, SAMPI:CAP0805, F.Cu at (244.9, 131.7)
- added C8: 2.2uF, SAMPI:CAP0603, F.Cu at (58.0, 111.2)
- added C9: 100pF, SAMPI:CAP0603, F.Cu at (58.0, 113.8)
- added D1: 2A/0.5VF, SAMPI:DO-214AC, F.Cu at (75.1, 139.6)
- added D2: 2A/0.5VF, SAMPI:DO-214AC, F.Cu at (75.1, 144.0)
- added D3: LOW BAT, SAMPI:LED0603, F.Cu at (61.7, 119.0)
- added D4: CHARGE, SAMPI:LED0603, F.Cu at (61.7, 121.6)
- added D5: APP, SAMPI:LED0603, F.Cu at (110.8, 53.4)
- added D6: TVS-5CH, SAMPI:SOT363, F.Cu at (99.7, 96.6)
- added D7: NB, SAMPI:LED0603, F.Cu at (79.4, 88.9)
- added D8: 2A/0.5VF, SAMPI:DO-214AC, F.Cu at (89.9, 121.1)
- added F1: 750mA/6.3V, SAMPI:FUSE1812, F.Cu at (67.3, 140.5)
- added FT1: 100R@100MHz, SAMPI:IND0805, F.Cu at (99.7, 93.0)
- added J1: USB, SAMPI:HDM-1x4x2.54-TH-RA, F.Cu at (46.9, 137.5)
- added J2: SOLAR, SAMPI:PAD02_2.54TH, F.Cu at (59.8, 136.0)
- added J3: PWR MONITOR, SAMPI:DIL04_2.54_MTHRA, F.Cu at (52.2, 128.2)
- added J4: RPDBG, SAMPI:DIL10_1.27_MTH, F.Cu at (109.4, 59.8)
- added J5: NANOSIM, SAMPI:SIM8051-6-0-14-01-A_GCT, F.Cu at (202.4, 54.5)
- added J6: DIL08, SAMPI:HDM-2x4x2.0-TH-RA, F.Cu at (250.3, 109.8)
- added J7: DIL08, SAMPI:HDM-2x4x2.0-TH-RA, F.Cu at (251.0, 100.7)
- added J8: DIL08, SAMPI:HDM-2x4x2.0-TH-RA, F.Cu at (236.9, 100.5)
- added L1: 2.2uH/3A, SAMPI:IND5852, F.Cu at (117.0, 90.3)
- added L2: 10uH/3A, SAMPI:IND7870, F.Cu at (108.9, 91.3)
- added L3: 47nH, SAMPI:IND0603, F.Cu at (79.4, 91.5)
- added L4: 10uH/3A, SAMPI:IND7870, F.Cu at (120.7, 77.5)
- added MD1: NB-IoT MODULE, SAMPI:xE310, F.Cu at (253.7, 59.8)
- added MD2: GPS ACTIVE ANTENNA, SAMPI:1575R-A, F.Cu at (239.9, 83.5)
- added Q1: MFET N, SAMPI:SOT23, F.Cu at (87.2, 90.9)
- added Q2: MFET N, SAMPI:SOT23, F.Cu at (91.8, 90.9)
- added R1: 1K, SAMPI:RES0603, F.Cu at (65.4, 103.4)
- added R10: 1K, SAMPI:RES0603, F.Cu at (69.1, 106.0)
- added R11: 53.6K, 1%, SAMPI:RES0603, F.Cu at (69.1, 108.6)
- added R12: 10K, 1%, SAMPI:RES0603, F.Cu at (69.1, 111.2)
- added R13: 1K, SAMPI:RES0603, F.Cu at (69.1, 113.8)
- added R14: 1K, SAMPI:RES0603, F.Cu at (69.1, 116.4)
- added R15: 1K, SAMPI:RES0603, F.Cu at (69.1, 119.0)
- added R16: 10K, 1%, SAMPI:RES0603, F.Cu at (69.1, 121.6)
- added R17: 100K, 1%, SAMPI:RES0603, F.Cu at (72.8, 103.4)
- added R18: 10K, 1%, SAMPI:RES0603, F.Cu at (72.8, 106.0)
- added R19: 680K, 1%, SAMPI:RES0603, F.Cu at (72.8, 108.6)
- added R2: 5.1K, 1%, SAMPI:RES0603, F.Cu at (65.4, 106.0)
- added R20: 10K, 1%, SAMPI:RES0603, F.Cu at (72.8, 111.2)
- added R21: 0R, SAMPI:RES0603, F.Cu at (72.8, 113.8)
- added R22: 10K, 1%, SAMPI:RES0603, F.Cu at (72.8, 116.4)
- added R23: 5.1K, 1%, SAMPI:RES0603, F.Cu at (110.8, 56.0)
- added R24: 5.1K, 1%, SAMPI:RES0603, F.Cu at (114.5, 42.9)
- added R25: 10K, 1%, SAMPI:RES0603, F.Cu at (114.5, 45.5)
- added R26: 1K, SAMPI:RES0603, F.Cu at (114.5, 48.1)
- added R27: 0R, SAMPI:RES0603, F.Cu at (114.5, 50.8)
- added R28: 1K, SAMPI:RES0603, F.Cu at (114.5, 53.4)
- added R29: 0R, SAMPI:RES0603, F.Cu at (79.4, 94.2)
- added R3: 10K, 1%, SAMPI:RES0603, F.Cu at (65.4, 108.6)
- added R30: 10K, 1%, SAMPI:RES0603, F.Cu at (83.1, 75.9)
- added R31: 1K, SAMPI:RES0603, F.Cu at (83.1, 78.5)
- added R32: 1K, SAMPI:RES0603, F.Cu at (83.1, 81.1)
- added R33: 150R, SAMPI:RES0603, F.Cu at (234.1, 125.3)
- added R34: 75K, 1%, SAMPI:RES0603, F.Cu at (83.1, 86.3)
- added R35: 10K, 1%, SAMPI:RES0603, F.Cu at (101.0, 108.6)
- added R36: 1K, SAMPI:RES0603, F.Cu at (244.9, 136.9)
- added R37: 150K, 1%, SAMPI:RES0603, F.Cu at (101.0, 113.8)
- added R38: 150K, 1%, SAMPI:RES0603, F.Cu at (104.7, 103.4)
- added R4: 10K, 1%, SAMPI:RES0603, F.Cu at (65.4, 111.2)
- added R5: 5.1K, 1%, SAMPI:RES0603, F.Cu at (65.4, 113.8)
- added R6: 1K, SAMPI:RES0603, F.Cu at (65.4, 116.4)
- added R7: 75K, 1%, SAMPI:RES0603, F.Cu at (65.4, 119.0)
- added R8: 36K, 1%, SAMPI:RES0603, F.Cu at (65.4, 121.6)
- added R9: 10K, 1%, SAMPI:RES0603, F.Cu at (69.1, 103.4)
- added TP1: VUSB, SAMPI:TP1MM, F.Cu at (73.1, 124.8)
- added TP10: VBOOST, SAMPI:TP1MM, F.Cu at (106.7, 116.9)
- added TP2: VNB, SAMPI:TP1MM, F.Cu at (73.1, 128.4)
- added TP3: 5V, SAMPI:TP1MM, F.Cu at (73.1, 132.0)
- added TP4: 3V3, SAMPI:TP1MM, F.Cu at (73.1, 135.6)
- added TP5: VBAT, SAMPI:TP1MM, F.Cu at (76.7, 124.8)
- added TP6: GND, SAMPI:TP1MM, F.Cu at (76.7, 128.4)
- added TP7: VDD, SAMPI:TP1MM, F.Cu at (76.7, 132.0)
- added TP8: 1V8, SAMPI:TP1MM, F.Cu at (96.0, 90.3)
- added TP9: VLNA, SAMPI:TP1MM, F.Cu at (96.0, 93.9)
- added U1: BUCK 5V, SAMPI:SOT-23-6_MCHP, F.Cu at (80.9, 125.7)
- added U10: LDO 3.3V/300mA, SAMPI:SOT-23-5_MCHP, F.Cu at (96.7, 77.3)
- added U11: DUST SENSOR CONNECTOR, SAMPI:HDM-6x1.5-SMD-RA, F.Cu at (238.2, 111.6)
- added U12: HUMI & TEMP, SAMPI:SHT4x, F.Cu at (238.1, 120.8)
- added U13: BOOST 5V, SAMPI:SOT-23-6_MCHP, F.Cu at (97.8, 117.9)
- added U14: DPS368, SAMPI:DPS368, F.Cu at (246.5, 143.1)
- added U2: BUCK-BOOST 3.8V, SAMPI:PowerVQFN15_TI, F.Cu at (106.6, 98.6)
- added U3: IDEAL DIODE, SAMPI:SOT363, F.Cu at (80.5, 135.3)
- added U4: MCP73871, SAMPI:VQFN20-4x4_MCHP, F.Cu at (116.7, 97.3)
- added U5: MCP1700, SAMPI:SOT23, F.Cu at (80.8, 130.8)
- added U6: SPI Memory, SAMPI:SOIC8_3.9_MCHP, F.Cu at (119.6, 59.0)
- added U7: PIC32MM MCU, SAMPI:TQFP48-7x7_MCHP, F.Cu at (221.8, 97.0)
- added U8: LEVEL SHIFT 1-CH, SAMPI:SOT-23-6_MCHP, F.Cu at (87.3, 77.3)
- added U9: LEVEL SHIFT 1-CH, SAMPI:SOT-23-6_MCHP, F.Cu at (92.0, 77.3)
- added X1: 32.768kHz, SAMPI:SMD4-7015, F.Cu at (135.2, 54.2)
- added Z1: 0R, SAMPI:RES0603, F.Cu at (249.8, 47.9)
Other:
- board size 73.2 x 82.3 mm -> 70 x 64.7 mm
