File: Hardware/WeatherStation.kicad_sch (KiCad schematic)
At the start: 0 parts

Commit message: UPDATE HARDWARE
UPDATE
Other:
- note added: "Analog signals"
- note added: "Digital signals"
Changed lines of the file:
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@@
+		)
+	)
+	(rectangle
+		(start 82.55 109.855)
+		(end 84.455 111.76)
+		(stroke
+			(width 0)
+			(type default)
+			(color 0 200 0 1)
+		)
+		(fill
+			(type color)
+			(color 0 200 0 1)
+		)
+	)
+	(rectangle
+		(start 82.55 113.03)
+		(end 84.455 114.935)
+		(stroke
+			(width 0)
+			(type default)
+			(color 114 86 0 1)
+		)
+		(fill
+			(type color)
+			(color 114 86 0 1)
 		)
 	)
@@
 		)
 	)
+	(text "Digital signals"
+		(exclude_from_sim no)
+		(at 91.44 114.3 0)
+		(effects
+			(font
+				(size 1.016 1.016)
+			)
+		)
+	)
 	(text "Internal connections"
 		(exclude_from_sim no)
@@
 	(text "3V3"
 		(exclude_from_sim no)
-		(at 148.844 112.268 0)
+		(at 149.225 112.395 0)
 		(effects
 			(font
@@
 	(text "5V,\n3.8V,\n3V3"
 		(exclude_from_sim no)
-		(at 103.124 81.026 0)
+		(at 102.87 80.645 0)
 		(effects
 			(font
@@
 				(size 1.016 1.016)
 			)
+		)
+	)
+	(text "Analog signals"
+		(exclude_from_sim no)
+		(at 90.805 111.125 0)
+		(effects
+			(font
+				(size 1.016 1.016)
+			)
