File: Hardware/MCU.kicad_sch (KiCad schematic)
At the start: 24 parts, among them J4 RPDBG, U6 SPI Memory, U7 PIC32MM MCU, X1 32.768kHz

Commit message: UPDATE HARDWARE
UPDATE
Parts:
- removed BT1: RESET, symbol SAMPI:BT
- removed BT2: APP, symbol SAMPI:BT
- added BT1: RESET, SAMPI:SW_SMD2_6.0x3.5, symbol SAMPI:BT3
- added BT2: APP, SAMPI:SW_SMD2_6.0x3.5, symbol SAMPI:BT3
- C30: MFT Samsung -> Samsung
- J4: footprint (none) -> SAMPI:DIL10_1.27_MTH
Connections:
- net +3.3V: now also J4.4 (VDD); no longer J4.3 (VDD)
- net DBG_RXD: now also J4.3 (DBG_RX), U7.26 (TDI/AN11/C1INA/RP9/SCL2/OCM2F/RB3); no longer J4.4 (DBG_RX)
- net DBG_TXD: now also J4.1 (DBG_TXD), U7.25 (AN4/C1INB/RP8/SDA2/OCM2E/RB2); no longer J4.2 (DBG_TXD)
- net GND: now also J4.6 (GND), BT1.2, BT2.2; no longer J4.5 (GND)
- net NB_DN: now also J4.7 (USB_DM); no longer J4.8 (USB_DM)
- net NB_DP: now also J4.5 (USB_DP); no longer J4.6 (USB_DP)
- net NB_VBUS: now also J4.9 (USB_VBUS); no longer J4.10 (USB_VBUS)
- net PGC: now also J4.10 (PGC), U7.24 (PGEC1/AN3/C1INC/C2INA/RP7/OCM2D/RB1); no longer J4.9 (PGC)
- net PGD: now also J4.8 (PGD/UPDI), U7.23 (PGED1/AN2/C1IND/C2INB/C3INC/RP6/RB0); no longer J4.7 (PGD/UPDI)
- net SOSCI: now also U7.35 (SOSCI/AN7/RP10/OCM3C/RB4)
- net SOSCO: now also U7.36 (SOSCO/SCLKI/RP5/PWRLCLK/OCM3D/RA4)
- net USB_DN: now also U7.9 (D-/RB10)
- net USB_DP: now also U7.10 (D+/RB11)
- net VBUS_SEN: now also U7.46 (VBUS/RB6)
- net ~{BT_APP}: now also BT2.1
- net ~{MCLR}: now also J4.2 (~{RESET}), U7.19 (~{MCLR}), BT1.1; no longer J4.1 (~{RESET})
- no-connect marks 6 -> 0

Commit message: UPDATE _FOOTPRINT
UPDATE
Parts:
- removed X1: 32.768kHz, SAMPI:SMD4-7015, symbol SAMPI:XTAL-2P
- added X1: 32.768kHz, SAMPI:SMD4-7015, symbol SAMPI:XTAL-4P
- U7: footprint (none) -> SAMPI:TQFP48-7x7_MCHP
- renumbered R23 to R21, R24 to R22, R25 to R23, R26 to R24, R27 to R25, R28 to R26
Connections:
- net GND: now also X1.2 (GND1), X1.3 (GND2)
- net SOSCI: now also X1.1 (X1)
- net SOSCO: now also X1.4 (X2)

Commit message: Update check BoM
update BoM
Parts:
- BT1, BT2, C27, C28, C29, C30, C31, C32, C33, C34, C35, C36, C37, D5, J4, R21, R22, R23, R24, R25, R26: Check (none) -> oke
Changed lines of the file:
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@@
 			)
 		)
-		(property "Check" ""
+		(property "Check" "oke"
 			(at 216.535 85.725 0)
 			(effects
@@
 			)
 		)
-		(property "Check" ""
+		(property "Check" "oke"
 			(at 212.725 67.31 0)
 			(effects
@@
 			)
 		)
-		(property "Check" ""
+		(property "Check" "oke"
 			(at 210.82 152.4 0)
 			(effects
@@
 			)
 		)
-		(property "Check" ""
+		(property "Check" "oke"
 			(at 180.34 116.84 0)
 			(effects
@@
 			)
 		)
-		(property "Check" ""
+		(property "Check" "oke"
 			(at 171.45 152.4 0)
 			(effects
@@
 			)
 		)
-		(property "Check" ""
+		(property "Check" "oke"
 			(at 224.155 154.305 0)
 			(effects
@@
 			)
 		)
-		(property "Check" ""
+		(property "Check" "oke"
 			(at 158.75 152.4 0)
 			(effects
@@
 			)
 		)
-		(property "Check" ""
+		(property "Check" "oke"
 			(at 191.135 142.24 0)
 			(effects
@@
 			)
 		)
-		(property "Check" ""
+		(property "Check" "oke"
 			(at 176.53 114.3 0)
 			(effects
@@
 			)
 		)
-		(property "Check" ""
+		(property "Check" "oke"
 			(at 213.995 105.41 0)
 			(effects
@@
 			)
 		)
-		(property "Check" ""
+		(property "Check" "oke"
 			(at 185.42 152.4 0)
 			(effects
@@
 			)
 		)
-		(property "Check" ""
+		(property "Check" "oke"
 			(at 232.41 144.78 0)
 			(effects
@@
 			)
 		)
-		(property "Check" ""
+		(property "Check" "oke"
 			(at 203.835 85.725 0)
 			(effects
@@
 			)
 		)
-		(property "Check" ""
+		(property "Check" "oke"
 			(at 222.25 105.41 0)
 			(effects
@@
 			)
 		)
-		(property "Check" ""
+		(property "Check" "oke"
 			(at 170.18 116.84 0)
 			(effects
@@
 			)
 		)
-		(property "Check" ""
+		(property "Check" "oke"
 			(at 194.31 114.3 0)
 			(effects
@@
 			)
 		)
-		(property "Check" ""
+		(property "Check" "oke"
 			(at 240.03 153.035 0)
 			(effects
@@
 			)
 		)
-		(property "Check" ""
+		(property "Check" "oke"
 			(at 198.755 154.305 0)
 			(effects
@@
 			)
 		)
-		(property "Check" ""
+		(property "Check" "oke"
 			(at 216.535 142.24 0)
 			(effects
@@
 			)
 		)
-		(property "Check" ""
+		(property "Check" "oke"
 			(at 205.74 105.41 0)
 			(effects
@@
 			)
 		)
-		(property "Check" ""
+		(property "Check" "oke"
 			(at 143.51 152.4 0)
 			(effects
