File: Hardware/NBMODULE.kicad_sch (KiCad schematic)
At the start: 50 parts, among them J5 NANOSIM, Q1 MFET N, Q2 MFET N, U10 LDO 3.3V/300mA, U8 LEVEL SHIFT 1-CH, U9 LEVEL SHIFT 1-CH

Commit message: UPDATE HARDWARE
UPDATE
Parts:
- ANT1: footprint (none) -> SAMPI:AH3G.303
- ANT2: footprint (none) -> SAMPI:U.FL
- C49: footprint (none) -> SAMPI:CAP_ELEC-6.6x6.6-DIA6.3
- C57, C58: footprint (none) -> SAMPI:SCAP1320
- C62: MFT Samsung -> Samsung
Changed lines of the file:
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@@
 			)
 		)
-		(property "Footprint" ""
+		(property "Footprint" "SAMPI:U.FL"
 			(at 217.17 58.42 0)
 			(effects
@@
 			)
 		)
-		(property "Footprint" ""
+		(property "Footprint" "SAMPI:CAP_ELEC-6.6x6.6-DIA6.3"
 			(at 180.34 109.855 0)
 			(effects
@@
 			)
 		)
-		(property "MFT" " Samsung"
+		(property "MFT" "Samsung"
 			(at 271.145 53.975 0)
 			(effects
@@
 			)
 		)
-		(property "Footprint" ""
+		(property "Footprint" "SAMPI:SCAP1320"
 			(at 226.06 114.935 0)
 			(effects
@@
 			)
 		)
-		(property "Footprint" ""
+		(property "Footprint" "SAMPI:SCAP1320"
 			(at 226.06 107.315 0)
 			(effects
@@
 			)
 		)
-		(property "Footprint" ""
+		(property "Footprint" "SAMPI:AH3G.303"
 			(at 196.215 51.435 0)
 			(effects

Commit message: UPDATE _FOOTPRINT
UPDATE
Parts:
- removed Z1, Z3: Cx, SAMPI:CAP0603, symbol SAMPI:CERCAP
- C49: footprint SAMPI:CAP_ELEC-6.6x6.6-DIA6.3 -> SAMPI:CAP2312-6032; MFT Aishi -> AVX; MNP EMK1CM221E83D00R -> TAJC227K006RNJ; Price 0.039 -> 0.241; Stock Link https://www.thegioiic.com/tu-nhom-smd-220uf-16v-6-3x7-7mm -> https://www.thegioiic.com/tu-tantalum-220uf-6-3v-2312-tajc2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
- J5: footprint (none) -> SAMPI:SIM8051-6-0-14-01-A_GCT
- MD1: value ME310G1 -> NB-IoT MODULE; footprint (none) -> SAMPI:xE310
- TP8, TP9: footprint (none) -> SAMPI:TP1MM; now fitted; now left out of the parts list
- renumbered R29 to R27, R30 to R28, R31 to R29, R32 to R30, R33 to R31, R34 to R32, Z2 to Z1
Connections:
- net +1V8: now also MD1.N16 (~{ONOFF}/~{WAKE}); no longer MD1.R1 (PWRMON)
- net at C50.2, C52.1, FT1.1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: now also MD1.AA3 (VBATT)
- net at Q2.3 (D): now also MD1.R1 (PWRMON); no longer MD1.N16 (~{ONOFF}/~{WAKE})
Other:
- moved on the sheet: Z1

Commit message: Update check BoM
update BoM
Parts:
- ANT1, ANT2, C38, C39, C40, C41, C42, C43, C44, C45, C46, C47, C48, C49, C50, C51, C52, C53, C54, C55, C56, C57, C58, C59, C60, C61, C62, D6, D7, FT1, J5, L3, MD1, MD2, Q1, Q2, R27, R28, R29, R30, R31, R32, Z1: Check (none) -> oke
Changed lines of the file:
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@@
 			)
 		)
-		(property "Check" ""
+		(property "Check" "oke"
 			(at 218.44 53.975 0)
 			(effects
@@
 			)
 		)
-		(property "Check" ""
+		(property "Check" "oke"
 			(at 198.755 109.855 0)
 			(effects
@@
 			)
 		)
-		(property "Check" ""
+		(property "Check" "oke"
 			(at 215.9 35.56 0)
 			(effects
@@
 			)
 		)
-		(property "Check" ""
+		(property "Check" "oke"
 			(at 71.12 76.2 0)
 			(effects
@@
 			)
 		)
-		(property "Check" ""
+		(property "Check" "oke"
 			(at 208.915 109.855 0)
 			(effects
@@
 			)
 		)
-		(property "Check" ""
+		(property "Check" "oke"
 			(at 180.34 109.855 0)
 			(effects
@@
 			)
 		)
-		(property "Check" ""
+		(property "Check" "oke"
 			(at 172.085 109.855 0)
 			(effects
@@
 			)
 		)
-		(property "Check" ""
+		(property "Check" "oke"
 			(at 42.545 77.47 0)
 			(effects
@@
 			)
 		)
-		(property "Check" ""
+		(property "Check" "oke"
 			(at 219.71 45.085 0)
 			(effects
@@
 			)
 		)
-		(property "Check" ""
+		(property "Check" "oke"
 			(at 206.375 89.535 0)
 			(effects
@@
 			)
 		)
-		(property "Check" ""
+		(property "Check" "oke"
 			(at 205.74 45.085 0)
 			(effects
@@
 			)
 		)
-		(property "Check" ""
+		(property "Check" "oke"
 			(at 102.235 162.56 0)
 			(effects
@@
 			)
 		)
-		(property "Check" ""
+		(property "Check" "oke"
 			(at 251.46 9.525 0)
 			(effects
@@
 			)
 		)
-		(property "Check" ""
+		(property "Check" "oke"
 			(at 212.09 112.395 0)
 			(effects
@@
 			)
 		)
-		(property "Check" ""
+		(property "Check" "oke"
 			(at 33.655 156.21 0)
 			(effects
@@
 			)
 		)
-		(property "Check" ""
+		(property "Check" "oke"
 			(at 173.99 74.295 0)
 			(effects
@@
 			)
 		)
-		(property "Check" ""
+		(property "Check" "oke"
 			(at 182.245 68.58 0)
 			(effects
@@
 			)
 		)
-		(property "Check" ""
+		(property "Check" "oke"
 			(at 88.9 185.42 0)
 			(effects
@@
 			)
 		)
-		(property "Check" ""
+		(property "Check" "oke"
 			(at 200.66 99.695 0)
 			(effects
@@
 			)
 		)
-		(property "Check" ""
+		(property "Check" "oke"
 			(at 228.6 53.975 0)
 			(effects
@@
 			)
 		)
-		(property "Check" ""
+		(property "Check" "oke"
 			(at 271.145 53.975 0)
 			(effects
@@
 			)
 		)
-		(property "Check" ""
+		(property "Check" "oke"
 			(at 56.515 162.56 0)
 			(effects
@@
 			)
 		)
-		(property "Check" ""
+		(property "Check" "oke"
 			(at 226.06 114.935 0)
 			(effects
@@
 			)
 		)
-		(property "Check" ""
+		(property "Check" "oke"
 			(at 245.11 53.975 0)
 			(effects
@@
 			)
 		)
-		(property "Check" ""
+		(property "Check" "oke"
 			(at 69.85 45.085 0)
 			(effects
@@
 			)
 		)
-		(property "Check" ""
+		(property "Check" "oke"
 			(at 60.325 77.47 0)
 			(effects
@@
 			)
 		)
-		(property "Check" ""
+		(property "Check" "oke"
 			(at 68.58 163.83 0)
 			(effects
@@
 			)
 		)
-		(property "Check" ""
+		(property "Check" "oke"
 			(at 226.06 107.315 0)
 			(effects
@@
 			)
 		)
-		(property "Check" ""
+		(property "Check" "oke"
 			(at 86.995 51.435 0)
 			(effects
@@
 			)
 		)
-		(property "Check" ""
+		(property "Check" "oke"
 			(at 78.74 51.435 0)
 			(effects
@@
 			)
 		)
-		(property "Check" ""
+		(property "Check" "oke"
 			(at 180.34 61.595 0)
 			(effects
@@
 			)
 		)
-		(property "Check" ""
+		(property "Check" "oke"
 			(at 100.965 36.195 0)
 			(effects
@@
 			)
 		)
-		(property "Check" ""
+		(property "Check" "oke"
 			(at 42.545 162.56 0)
 			(effects
@@
 			)
 		)
-		(property "Check" ""
+		(property "Check" "oke"
 			(at 97.155 184.15 0)
 			(effects
@@
 			)
 		)
-		(property "Check" ""
+		(property "Check" "oke"
 			(at 194.945 28.575 0)
 			(effects
@@
 			)
 		)
-		(property "Check" ""
+		(property "Check" "oke"
 			(at 33.655 58.42 0)
 			(effects
@@
 			)
 		)
-		(property "Check" ""
+		(property "Check" "oke"
 			(at 51.435 77.47 0)
 			(effects
@@
 			)
 		)
-		(property "Check" ""
+		(property "Check" "oke"
 			(at 51.435 184.15 0)
 			(effects
@@
 			)
 		)
-		(property "Check" ""
+		(property "Check" "oke"
 			(at 182.245 29.845 0)
 			(effects
@@
 			)
 		)
-		(property "Check" ""
+		(property "Check" "oke"
 			(at 198.755 83.185 0)
 			(effects
@@
 			)
 		)
-		(property "Check" ""
+		(property "Check" "oke"
 			(at 231.775 56.515 0)
 			(effects
@@
 			)
 		)
-		(property "Check" ""
+		(property "Check" "oke"
 			(at 63.5 80.01 0)
 			(effects
@@
 			)
 		)
-		(property "Check" ""
+		(property "Check" "oke"
 			(at 184.785 112.395 0)
 			(effects
