File: Hardware/POWER.kicad_sch (KiCad schematic)
At the start: 72 parts, among them J1 USB C, J2 SOLAR, J3 PWR MONITOR, U1 BUCK 5V, U2 BUCK-BOOST 3.8V, U3 IDEAL DIODE, U4 MCP73871, U5 MCP1700

Commit message: UPDATE HARDWARE
UPDATE
Parts:
- BAT1, BAT2: footprint (none) -> SAMPI:PAD02_2.54TH
- C14, C18, C2, C21, C22, C24, C3, C7: MFT Samsung -> Samsung
- C19, C5: footprint (none) -> SAMPI:CAP_ELEC-6.6x6.6-DIA6.3
- C20, C26: footprint (none) -> SAMPI:CAP_ELEC-10.3x10.3-DIA10
- D1, D2: footprint (none) -> SAMPI:DO-214AC
- F1: value 1A -> 750mA/6.3V; footprint (none) -> SAMPI:FUSE1812
- J3: footprint (none) -> SAMPI:DIL04_2.54_MTHRA
Connections:
- net VBAT: no longer R21.1
- net at C21.1, J3.1, U4.14 (VBAT)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: now also R21.1
Other:
- moved on the sheet: C23, J3, R21, R22, TP5

Commit message: UPDATE _FOOTPRINT
UPDATE
Parts:
- removed J1: USB C, SAMPI:USB4105, symbol SAMPI:USB4105
- removed R1, R4: 5.1K, 1%, SAMPI:RES0603, symbol SAMPI:RES
- added J1: USB, SAMPI:HDM-1x4x2.54-TH-RA, symbol SAMPI:SIL04-1
- BAT1, BAT2: footprint SAMPI:PAD02_2.54TH -> SAMPI:BAT18650-PCBPAD
- C19: footprint SAMPI:CAP_ELEC-6.6x6.6-DIA6.3 -> SAMPI:CAP2312-6032; MFT Aishi -> AVX; MNP EMK1CM221E83D00R -> TAJC227K006RNJ; Price 0.039 -> 0.241; Stock Link https://www.thegioiic.com/tu-nhom-smd-220uf-16v-6-3x7-7mm -> https://www.thegioiic.com/tu-tantalum-220uf-6-3v-2312-tajc2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
- C20, C26: value 470uF -> 220uF; footprint SAMPI:CAP_ELEC-10.3x10.3-DIA10 -> SAMPI:CAP2312-6032; MFT Nichicon -> AVX; MNP UUD1E471MNL1GS -> TAJC227K006RNJ; Price 0.088 -> 0.241; Stock Link https://www.thegioiic.com/tu-nhom-smd-470uf-25v-10x10-5mm -> https://www.thegioiic.com/tu-tantalum-220uf-6-3v-2312-tajc2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
- C5: value 220uF -> 470uF; footprint SAMPI:CAP_ELEC-6.6x6.6-DIA6.3 -> SAMPI:CAP_ELEC-10.3x10.3-DIA10; MFT Aishi -> Nichicon; MNP EMK1CM221E83D00R -> UUD1E471MNL1GS; Price 0.039 -> 0.088; Stock Link https://www.thegioiic.com/tu-nhom-smd-220uf-16v-6-3x7-7mm -> https://www.thegioiic.com/tu-nhom-smd-470uf-25v-10x10-5mm
- J2: footprint PAD02_2.54TH -> SAMPI:PAD02_2.54TH
- L1: footprint (none) -> SAMPI:IND5852
- L2: footprint (none) -> SAMPI:IND7870
- TP1, TP2, TP3, TP4, TP5, TP6, TP7: footprint (none) -> SAMPI:TP1MM; now fitted; now left out of the parts list
- U2: footprint (none) -> SAMPI:PowerVQFN15_TI
- U4: footprint (none) -> SAMPI:VQFN20-4x4_MCHP
- renumbered R2 to R1, R12 to R10, R13 to R11, R14 to R12, R15 to R13, R16 to R14, R17 to R15, R18 to R16, R19 to R17, R20 to R18, R21 to R19, R3 to R2, R22 to R20, R5 to R3, R6 to R4, R7 to R5, R8 to R6, R9 to R7, R10 to R8, R11 to R9
Connections:
- net GND: now also BAT1.-, BAT2.-, J1.1; no longer BAT1.2 (-), BAT2.2 (-)
- net USB_DN: now also J1.3
- net USB_DP: now also J1.2
- net VBAT: now also BAT1.+, BAT2.+; no longer BAT1.1 (+), BAT2.1 (+)
- net at F1.1: now also J1.4
- no-connect marks 3 -> 1
Other:
- moved on the sheet: F1

Commit message: Update check BoM
update BoM
Parts:
- BAT1, BAT2, C1, C10, C11, C12, C13, C14, C15, C16, C17, C18, C19, C2, C20, C21, C22, C23, C24, C25, C26, C3, C4, C5, C6, C7, C8, C9, D1, D2, D3, D4, F1, J1, J2, J3, L1, L2, R1, R10, R11, R12, R13, R14, R15, R16, R17, R18, R19, R2, R20, R3, R4, R5, R6, R7, R8, R9: Check (none) -> oke
Changed lines of the file:
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@@
 			)
 		)
-		(property "Check" ""
+		(property "Check" "oke"
 			(at 129.54 141.605 0)
 			(effects
@@
 			)
 		)
-		(property "Check" ""
+		(property "Check" "oke"
 			(at 264.16 29.21 0)
 			(effects
@@
 			)
 		)
-		(property "Check" ""
+		(property "Check" "oke"
 			(at 156.21 86.995 0)
 			(effects
@@
 			)
 		)
-		(property "Check" ""
+		(property "Check" "oke"
 			(at 132.715 86.995 0)
 			(effects
@@
 			)
 		)
-		(property "Check" ""
+		(property "Check" "oke"
 			(at 62.865 104.775 0)
 			(effects
@@
 			)
 		)
-		(property "Check" ""
+		(property "Check" "oke"
 			(at 156.845 131.445 0)
 			(effects
@@
 			)
 		)
-		(property "Check" ""
+		(property "Check" "oke"
 			(at 188.595 40.64 0)
 			(effects
@@
 			)
 		)
-		(property "Check" ""
+		(property "Check" "oke"
 			(at 73.66 114.935 0)
 			(effects
@@
 			)
 		)
-		(property "Check" ""
+		(property "Check" "oke"
 			(at 128.27 140.335 0)
 			(effects
@@
 			)
 		)
-		(property "Check" ""
+		(property "Check" "oke"
 			(at 126.365 29.21 0)
 			(effects
@@
 			)
 		)
-		(property "Check" ""
+		(property "Check" "oke"
 			(at 197.485 86.995 0)
 			(effects
@@
 			)
 		)
-		(property "Check" ""
+		(property "Check" "oke"
 			(at 101.6 86.995 0)
 			(effects
@@
 			)
 		)
-		(property "Check" ""
+		(property "Check" "oke"
 			(at 188.595 50.8 0)
 			(effects
@@
 			)
 		)
-		(property "Check" ""
+		(property "Check" "oke"
 			(at 222.25 86.995 0)
 			(effects
@@
 			)
 		)
-		(property "Check" ""
+		(property "Check" "oke"
 			(at 54.61 131.445 0)
 			(effects
@@
 			)
 		)
-		(property "Check" ""
+		(property "Check" "oke"
 			(at 203.2 46.99 0)
 			(effects
@@
 			)
 		)
-		(property "Check" ""
+		(property "Check" "oke"
 			(at 203.2 36.83 0)
 			(effects
@@
 			)
 		)
-		(property "Check" ""
+		(property "Check" "oke"
 			(at 54.61 151.765 0)
 			(effects
@@
 			)
 		)
-		(property "Check" ""
+		(property "Check" "oke"
 			(at 111.76 78.105 0)
 			(effects
@@
 			)
 		)
-		(property "Check" ""
+		(property "Check" "oke"
 			(at 116.84 98.425 0)
 			(effects
@@
 			)
 		)
-		(property "Check" ""
+		(property "Check" "oke"
 			(at 105.41 47.625 0)
 			(effects
@@
 			)
 		)
-		(property "Check" ""
+		(property "Check" "oke"
 			(at 243.84 35.56 0)
 			(effects
@@
 			)
 		)
-		(property "Check" ""
+		(property "Check" "oke"
 			(at 88.9 29.21 0)
 			(effects
@@
 			)
 		)
-		(property "Check" ""
+		(property "Check" "oke"
 			(at 163.195 40.64 0)
 			(effects
@@
 			)
 		)
-		(property "Check" ""
+		(property "Check" "oke"
 			(at 167.005 86.995 0)
 			(effects
@@
 			)
 		)
-		(property "Check" ""
+		(property "Check" "oke"
 			(at 74.295 104.775 0)
 			(effects
@@
 			)
 		)
-		(property "Check" ""
+		(property "Check" "oke"
 			(at 137.795 98.425 0)
 			(effects
@@
 			)
 		)
-		(property "Check" ""
+		(property "Check" "oke"
 			(at 197.485 36.83 0)
 			(effects
@@
 			)
 		)
-		(property "Check" ""
+		(property "Check" "oke"
 			(at 132.715 99.695 0)
 			(effects
@@
 			)
 		)
-		(property "Check" ""
+		(property "Check" "oke"
 			(at 165.735 131.445 0)
 			(effects
@@
 			)
 		)
-		(property "Check" ""
+		(property "Check" "oke"
 			(at 275.59 29.21 0)
 			(effects
@@
 			)
 		)
-		(property "Check" ""
+		(property "Check" "oke"
 			(at 54.61 86.995 0)
 			(effects
@@
 			)
 		)
-		(property "Check" ""
+		(property "Check" "oke"
 			(at 69.215 89.535 0)
 			(effects
@@
 			)
 		)
-		(property "Check" ""
+		(property "Check" "oke"
 			(at 137.16 29.21 0)
 			(effects
@@
 			)
 		)
-		(property "Check" ""
+		(property "Check" "oke"
 			(at 46.355 35.56 0)
 			(effects
@@
 			)
 		)
-		(property "Check" ""
+		(property "Check" "oke"
 			(at 123.19 131.445 0)
 			(effects
@@
 			)
 		)
-		(property "Check" ""
+		(property "Check" "oke"
 			(at 64.135 22.86 0)
 			(effects
@@
 			)
 		)
-		(property "Check" ""
+		(property "Check" "oke"
 			(at 146.685 131.445 0)
 			(effects
@@
 			)
 		)
-		(property "Check" ""
+		(property "Check" "oke"
 			(at 139.065 99.695 0)
 			(effects
@@
 			)
 		)
-		(property "Check" ""
+		(property "Check" "oke"
 			(at 212.725 46.99 0)
 			(effects
@@
 			)
 		)
-		(property "Check" ""
+		(property "Check" "oke"
 			(at 123.19 86.995 0)
 			(effects
@@
 			)
 		)
-		(property "Check" ""
+		(property "Check" "oke"
 			(at 78.74 29.21 0)
 			(effects
@@
 			)
 		)
-		(property "Check" ""
+		(property "Check" "oke"
 			(at 48.895 79.375 0)
 			(effects
@@
 			)
 		)
-		(property "Check" ""
+		(property "Check" "oke"
 			(at 99.06 40.005 0)
 			(effects
@@
 			)
 		)
-		(property "Check" ""
+		(property "Check" "oke"
 			(at 159.385 32.385 0)
 			(effects
@@
 			)
 		)
-		(property "Check" ""
+		(property "Check" "oke"
 			(at 99.06 122.555 0)
 			(effects
@@
 			)
 		)
-		(property "Check" ""
+		(property "Check" "oke"
 			(at 64.135 103.505 0)
 			(effects
@@
 			)
 		)
-		(property "Check" ""
+		(property "Check" "oke"
 			(at 143.51 43.18 0)
 			(effects
@@
 			)
 		)
-		(property "Check" ""
+		(property "Check" "oke"
 			(at 93.98 47.625 0)
 			(effects
@@
 			)
 		)
-		(property "Check" ""
+		(property "Check" "oke"
 			(at 123.19 141.605 0)
 			(effects
@@
 			)
 		)
-		(property "Check" ""
+		(property "Check" "oke"
 			(at 219.075 28.575 0)
 			(effects
@@
 			)
 		)
-		(property "Check" ""
+		(property "Check" "oke"
 			(at 104.14 46.355 0)
 			(effects
@@
 			)
 		)
-		(property "Check" ""
+		(property "Check" "oke"
 			(at 188.595 45.72 0)
 			(effects
@@
 			)
 		)
-		(property "Check" ""
+		(property "Check" "oke"
 			(at 256.54 35.56 0)
 			(effects
@@
 			)
 		)
-		(property "Check" ""
+		(property "Check" "oke"
 			(at 64.135 86.995 0)
 			(effects
@@
 			)
 		)
-		(property "Check" ""
+		(property "Check" "oke"
 			(at 113.665 131.445 0)
 			(effects
@@
 			)
 		)
-		(property "Check" ""
+		(property "Check" "oke"
 			(at 142.875 33.02 0)
 			(effects
@@
 			)
 		)
-		(property "Check" ""
+		(property "Check" "oke"
 			(at 100.33 78.105 0)
 			(effects
