File: Hardware/SENSORS.kicad_sch (KiCad schematic)
At the start: 30 parts, among them J6 DIL08, J7 DIL08, J8 DIL08, U11 DUST SENSOR, U12 HUMI & TEMP, U13 BOOST 5V, U14 BM1383

Commit message: UPDATE HARDWARE
UPDATE
Parts:
- removed C74: 2.2uF, SAMPI:CAP0603, symbol SAMPI:CERCAP
- removed U14: BM1383, symbol SAMPI:BM1383
- added CB1: CABLE, symbol SAMPI:CABLE
- added CB2: CABLE 2, symbol SAMPI:CABLE2
- added CB3: CABLE 3, symbol SAMPI:CABLE3
- added MD3: DUST SENSOR MODULE, symbol SAMPI:GP2Y1014AU_MODULE
- added U14: DPS368, SAMPI:DPS368, symbol SAMPI:DPS368
- C63, C64, C67, C76: MFT Samsung -> Samsung
- C65, C72: footprint (none) -> SAMPI:CAP_ELEC-6.6x6.6-DIA6.3
- D8: footprint (none) -> SAMPI:DO-214AC
- U11: value DUST SENSOR -> DUST SENSOR CONNECTOR; MFT SHARP -> JST; MNP GP2Y1014AU -> S6B-ZR-SM4A-TF; Price 4.079 -> 0.035; Stock Link https://www.thegioiic.com/gp2y1014au-cam-bien-bui-pm2-5 -> https://www.thegioiic.com/dau-zh-1-5mm-6-chan-dan-smd-nam-n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
- U12: MFT Sensirion -> Sensirion
Connections:
- net GND1: now also U14.1 (GND), U14.7 (GND)
- net SCL1: now also U14.4 (SDO)
- net SDA1: now also U14.3 (SDI/SDA)
- net VSEN1: now also U14.6 (VDDIO), U14.8 (VDD)
- no-connect marks 1 -> 2
Other:
- moved on the sheet: C64, C68, C70, C71, C72, C73, D8, J7, J8, L4, R36, R37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

Commit message: UPDATE _FOOTPRINT
UPDATE
Parts:
- C65, C72: footprint SAMPI:CAP_ELEC-6.6x6.6-DIA6.3 -> SAMPI:CAP2312-6032; MFT Aishi -> AVX; MNP EMK1CM221E83D00R -> TAJC227K006RNJ; Price 0.039 -> 0.241; Stock Link https://www.thegioiic.com/tu-nhom-smd-220uf-16v-6-3x7-7mm -> https://www.thegioiic.com/tu-tantalum-220uf-6-3v-2312-tajc2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
- CB1: value CABLE -> CABLE 6x1.5MM; MFT (none) -> OEM; MNP (none) -> ZH1.5-10CM; Price (none) -> 0.154; Stock Link (none) -> https://www.thegioiic.com/day-bus-zh1-5-cai-cai-6-tiep-diem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
- CB2: value CABLE 2 -> CABLE IDC-8x2MM-30CM; MFT (none) -> OEM; MNP (none) -> IDC8x2-30CM; Price (none) -> 1.009; Stock Link (none) -> https://www.thegioiic.com/day-cap-idc-cai-cai-cung-huong-8-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
- CB3: value CABLE 3 -> CABLE IDC-8x2MM-50CM; MFT (none) -> OEM; MNP (none) -> IDC8x2-50CM; Price (none) -> 1.228; Stock Link (none) -> https://www.thegioiic.com/day-cap-idc-cai-cai-cung-huong-8-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
- J6, J7, J8: footprint (none) -> SAMPI:HDM-2x4x2.0-TH-RA
- L4: footprint (none) -> SAMPI:IND7870
- TP10: footprint (none) -> SAMPI:TP1MM; now fitted; now left out of the parts list
- U11: footprint (none) -> SAMPI:HDM-6x1.5-SMD-RA
- U12: footprint (none) -> SAMPI:SHT4x
- renumbered C75 to C74, C76 to C75, R35 to R33, R36 to R34, R37 to R35, R38 to R36, R39 to R37, R40 to R38
Connections:
- net GND: no longer C67.2, C75.2
- net GND1: now also C67.2, C75.2, U11.7 (EP), U11.8 (EP)
Other:
- note removed: "IDC-8x2 CABLE"
- moved on the sheet: CB1, MD3

Commit message: Update check BoM
update BoM
Parts:
- C63, C64, C65, C66, C67, C68, C69, C70, C71, C72, C73, C74, C75, CB1, CB2, CB3, D8, J6, J7, J8, L4, MD3, R33, R34, R35, R36, R37, R38: Check (none) -> oke
Changed lines of the file:
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@@
 			)
 		)
-		(property "Check" ""
+		(property "Check" "oke"
 			(at 39.37 64.77 0)
 			(effects
@@
 			)
 		)
-		(property "Check" ""
+		(property "Check" "oke"
 			(at 53.34 39.37 0)
 			(effects
@@
 			)
 		)
-		(property "Check" ""
+		(property "Check" "oke"
 			(at 100.965 118.11 0)
 			(effects
@@
 			)
 		)
-		(property "Check" ""
+		(property "Check" "oke"
 			(at 40.64 102.235 0)
 			(effects
@@
 			)
 		)
-		(property "Check" ""
+		(property "Check" "oke"
 			(at 78.74 118.11 0)
 			(effects
@@
 			)
 		)
-		(property "Check" ""
+		(property "Check" "oke"
 			(at 137.795 139.7 0)
 			(effects
@@
 			)
 		)
-		(property "Check" ""
+		(property "Check" "oke"
 			(at 29.21 118.11 0)
 			(effects
@@
 			)
 		)
-		(property "Check" ""
+		(property "Check" "oke"
 			(at 91.44 118.11 0)
 			(effects
@@
 			)
 		)
-		(property "Check" ""
+		(property "Check" "oke"
 			(at 56.515 109.22 0)
 			(effects
@@
 			)
 		)
-		(property "Check" ""
+		(property "Check" "oke"
 			(at 136.525 113.665 0)
 			(effects
@@
 			)
 		)
-		(property "Check" ""
+		(property "Check" "oke"
 			(at 69.215 118.11 0)
 			(effects
@@
 			)
 		)
-		(property "Check" ""
+		(property "Check" "oke"
 			(at 123.19 109.22 0)
 			(effects
@@
 			)
 		)
-		(property "Check" ""
+		(property "Check" "oke"
 			(at 105.41 151.765 0)
 			(effects
@@
 			)
 		)
-		(property "Check" ""
+		(property "Check" "oke"
 			(at 58.42 80.645 0)
 			(effects
@@
 			)
 		)
-		(property "Check" ""
+		(property "Check" "oke"
 			(at 62.865 39.37 0)
 			(effects
@@
 			)
 		)
-		(property "Check" ""
+		(property "Check" "oke"
 			(at 123.19 135.255 0)
 			(effects
@@
 			)
 		)
-		(property "Check" ""
+		(property "Check" "oke"
 			(at 78.74 128.27 0)
 			(effects
@@
 			)
 		)
-		(property "Check" ""
+		(property "Check" "oke"
 			(at 115.57 53.34 0)
 			(effects
@@
 			)
 		)
-		(property "Check" ""
+		(property "Check" "oke"
 			(at 126.365 39.37 0)
 			(effects
@@
 			)
 		)
-		(property "Check" ""
+		(property "Check" "oke"
 			(at 79.375 60.96 0)
 			(effects
@@
 			)
 		)
-		(property "Check" ""
+		(property "Check" "oke"
 			(at 105.41 139.065 0)
 			(effects
@@
 			)
 		)
-		(property "Check" ""
+		(property "Check" "oke"
 			(at 93.345 139.065 0)
 			(effects
@@
 			)
 		)
-		(property "Check" ""
+		(property "Check" "oke"
 			(at 57.15 69.215 0)
 			(effects
@@
 			)
 		)
-		(property "Check" ""
+		(property "Check" "oke"
 			(at 116.205 39.37 0)
 			(effects
@@
 			)
 		)
-		(property "Check" ""
+		(property "Check" "oke"
 			(at 93.345 151.765 0)
 			(effects
@@
 			)
 		)
-		(property "Check" ""
+		(property "Check" "oke"
 			(at 30.48 58.42 0)
 			(effects
@@
 			)
 		)
-		(property "Check" ""
+		(property "Check" "oke"
 			(at 24.13 64.77 0)
 			(effects
@@
 			)
 		)
-		(property "Check" ""
+		(property "Check" "oke"
 			(at 80.645 62.23 0)
 			(effects
